Commit message: Fix: Resolve TF tree conflicts, correct sensor orientations, and fix IMU units
- Rotated Lidar and IMU frames by 180 degrees (yaw) in URDF to match physical mounting.
- Disabled 'enable_odom_tf' in diff_drive_controller to let EKF be the sole publisher of odom -> base_link.
- Fixed critical bug in MPU6050 driver: converted gyro output from deg/s to rad/s (REP-145 compliance) and added <cmath>.
- Disabled lateral velocity (vy) fusion in EKF config (non-holonomic constraint).
- Updated sensor_fusion launch file to load full mpu6050.yaml parameters.

File: src/warehouse_real_description/description/lidar.xacro (robot description, xacro)
@@ -7,5 +7,5 @@
         <parent link="chassis"/>
         <child link="laser_frame"/>
-        <origin xyz="0.363 0 0.0785" rpy="0 0 0"/>
+        <origin xyz="0.363 0 0.0785" rpy="0 0 3.14159"/>
     </joint>
     <link name="laser_frame">

File: src/warehouse_real_description/description/robot_core.xacro (robot description, xacro)
@@ -193,5 +193,5 @@
         <parent link="base_link"/>
         <child link="imu_link"/>
-        <origin xyz="0 0 0.05" rpy="0 0 0"/>
+        <origin xyz="0 0 0.05" rpy="0 0 3.14159"/>
     </joint>
     <link name="lifter_link">
